Commit message: Added required Gazebo simulaion infastructure

File: agv_pus_description/urdf/mech/agv_base.urdf.xacro (robot description, xacro)
@@ -17,5 +17,5 @@
         <visual>
             <geometry>
-                <mesh filename="package://agv_pus_description/meshes/vehicle/visual/base_link.STL"/>
+                <mesh filename="file://$(find agv_pus_description)/meshes/vehicle/visual/base_link.STL"/>
             </geometry>
             <material name="blue">

File: agv_pus_description/urdf/mech/mecanum_wheel.urdf.xacro (robot description, xacro)
@@ -1,5 +1,5 @@
 <?xml version="1.0"?>
 <robot xmlns:xacro="http://www.ros.org/wiki/xacro">
-  <xacro:property name="wheel_radius" value="0.1016" />
+  <xacro:property name="wheel_radius" value="0.1015" />
   <xacro:property name="wheel_separation" value="0.85519" />
   <xacro:property name="wheel_width" value="0.03899" />

File: agv_pus_description/urdf/robots/agv_pus.urdf.xacro (robot description, xacro)
@@ -1,4 +1,4 @@
 <?xml version="1.0"?>
-<robot xmlns:xacro="http://www.ros.org/wiki/xacro" name="rosmaster_x3">
+<robot xmlns:xacro="http://www.ros.org/wiki/xacro" name="agv_pus">
     <xacro:property name="M_PI" value="3.1415926535897931" />
     <xacro:arg name="robot_name" default="agv_pus"/>
@@ -49,13 +49,13 @@
       xyz_offset='0.437 0.0044 0.210'
       rpy_offset="0 0 0"/>
-    <!--xacro:include filename="$(find yahboom_rosmaster_description)/urdf/control/velocity_control_plugin.urdf.xacro" />
+    <xacro:include filename="$(find agv_pus_description)/urdf/control/velocity_control_plugin.urdf.xacro" />
     <xacro:load_velocity_control_plugin use_gazebo="$(arg use_gazebo)"/>
-    <xacro:include filename="$(find yahboom_rosmaster_description)/urdf/control/gazebo_sim_ros2_control.urdf.xacro" />
+    <xacro:include filename="$(find agv_pus_description)/urdf/control/gazebo_sim_ros2_control.urdf.xacro" />
     <xacro:load_gazebo_sim_ros2_control_plugin
       robot_name="$(arg robot_name)"
       use_gazebo="$(arg use_gazebo)"/>
-    <xacro:include filename="$(find yahboom_rosmaster_description)/urdf/control/rosmaster_x3_ros2_control.urdf.xacro" />
-    <xacro:yahboom_rosmaster_ros2_control
+    <xacro:include filename="$(find agv_pus_description)/urdf/control/rosmaster_x3_ros2_control.urdf.xacro" />
+    <xacro:agv_pus_ros2_control
       prefix="$(arg prefix)"
-      use_gazebo="$(arg use_gazebo)"/-->
+      use_gazebo="$(arg use_gazebo)"/>
 </robot>

Commit message: Added SLAM and debuged Lidar issues

File: agv_pus_description/urdf/mech/agv_base.urdf.xacro (robot description, xacro)
@@ -27,5 +27,5 @@
         <collision>
             <geometry>
-                <box size="${base_length} ${base_width} ${base_height}"/>
+                <box size="${base_length + 0.2} ${base_width} ${base_height}"/>
             </geometry>
             <origin xyz="0 0 ${base_height/2 - coordinate_z_offset}" rpy="0 0 0"/>

File: agv_pus_description/urdf/sensors/lidar.urdf.xacro (robot description, xacro)
@@ -2,4 +2,5 @@
 <robot xmlns:xacro="http://www.ros.org/wiki/xacro">
   <xacro:property name="M_PI" value="3.1415926535897931" />
+  <!-- Ta kurba vidi samega sebe, povecaj min_range, lahk ga pol ekzaktno dolocis -->
   <xacro:macro name="lidar_sensor" params="
     prefix:=''
@@ -26,7 +27,7 @@
     update_rate:=10
     ray_count:=720
-    min_angle:='-3.14159'
-    max_angle:='3.14159'
-    min_range:='0.20'
+    min_angle:='-3.14 '
+    max_angle:='3.14 '
+    min_range:='1.20'
     max_range:='30.0'
     range_resolution:='0.013'
